File: hardware/ambient-light-v3.kicad_pcb (KiCad board)
At the start: 2 copper layers, 25 x 15 mm, 24 parts, among them P1 CON-SENSOR2, P2 DEBUG, P3 BOOT, U1 XMC1XXX24, U2 LTR-329ALS, U3 DRILL, U4 DRILL, U5 DRILL, U6 DRILL

Commit message: Add logos
Parts:
- removed the VAL at (136.0, 94.0)
- added G***: LOGO, kicad-libraries:Logo_CoMCU, B.Cu at (142.4, 94.0)
- added VAL: WEEE_7mm, kicad-libraries:WEEE_7mm, B.Cu at (137.0, 94.3)
- moved VAL 0.20 mm to (149.2, 94.0), turned to 180 degrees
