File: hardware/ambient-light-v3.kicad_pcb (KiCad board)
At the start: 2 copper layers, 25 x 15 mm, 25 parts, among them P1 CON-SENSOR2, P2 DEBUG, P3 BOOT, U1 XMC1XXX24, U2 LTR-329ALS, U3 DRILL, U4 DRILL, U5 DRILL, U6 DRILL

Commit message: specify processor as xmc1100
Parts:
- U1: value XMC1XXX24 -> XMC1100
